Commit message: fix: improve RViz goal marker and clean node shutdown

File: src/drone_bringup/urdf/quadrotor.urdf (robot description, URDF)
Before this commit: robot quadrotor, 1 links, 0 joints
Links:
- added link body_link, mass 1.0; visual box size=0.08 0.06 0.035; visual box size=0.25 0.15 0.08
- link base_link: mass 1.0 -> None; geometry 
Joints:
- added joint base_to_body: type fixed, parent base_link, child body_link, origin xyz=0 0 0 rpy=0 0 0
